File: weird-generator-front-panel.kicad_pcb (KiCad board)
At the start: 2 copper layers, 100 x 205 mm, 25 parts

Commit message: Completed design
Parts:
- removed the ? at (104.6, 47.3)
- removed the ? at (76.0, 47.3)
- removed the REF** at (82.5, 79.5)
- removed the REF** at (118.4, 69.8)
- removed the REF** at (62.0, 69.8)
- removed the REF** at (45.0, 235.0)
- removed the REF** at (82.5, 113.3)
- removed the REF** at (90.0, 212.7)
- removed the REF** at (45.0, 40.0)
- removed the REF** at (118.4, 103.8)
- removed the REF** at (62.0, 171.8)
- removed the REF** at (98.3, 147.1)
- removed the REF** at (98.3, 113.3)
- removed the REF** at (118.4, 171.8)
- removed the REF** at (62.0, 103.8)
- removed the REF** at (62.0, 137.8)
- removed the REF** at (75.8, 227.8)
- removed the REF** at (104.4, 227.8)
- removed the REF** at (82.5, 147.1)
- removed the REF** at (118.4, 137.8)
- removed the REF** at (61.6, 212.7)
- removed the REF** at (135.0, 235.0)
- removed the REF** at (135.0, 40.0)
- removed the REF** at (118.4, 212.7)
- removed the REF** at (98.3, 79.5)
- added ?: , , F.Cu at (136.8, 112.4)
- added ?: , , F.Cu at (153.8, 112.4)
- added ?: , , F.Cu at (128.3, 202.4)
- added ?: , , F.Cu at (170.8, 112.4)
- added ?: , , F.Cu at (136.8, 202.4)
- added ?: , , F.Cu at (170.8, 202.4)
- added ?: , , F.Cu at (128.4, 48.1)
- added ?: , , F.Cu at (145.3, 112.4)
- added ?: , , F.Cu at (145.3, 202.4)
- added ?: , , F.Cu at (136.9, 48.1)
- added ?: , , F.Cu at (162.4, 48.1)
- added ?: , , F.Cu at (145.4, 48.1)
- added ?: , , F.Cu at (162.3, 112.4)
- added ?: , , F.Cu at (162.3, 202.4)
- added ?: , , F.Cu at (153.9, 48.1)
- added ?: , , F.Cu at (170.9, 48.1)
- added ?: , , F.Cu at (128.3, 112.4)
- added ?: , , F.Cu at (153.8, 202.4)
- added REF**: sw_fx_panel_small, fx_synth_parts:sw_fx_panel_small, F.Cu at (126.5, 192.0)
- added REF**: pot_fx_panel_small_knob_1, fx_synth_parts:pot_fx_panel_small_knob_1, F.Cu at (149.6, 157.0)
- added REF**: MountingHole_3.2mm_M3_ISO14580_Pad, MountingHole:MountingHole_3.2mm_M3_ISO14580_Pad, F.Cu at (214.5, 206.0)
- added REF**: sw_fx_panel_small, fx_synth_parts:sw_fx_panel_small, F.Cu at (168.8, 98.4)
- added REF**: pot_fx_panel_small_knob_1, fx_synth_parts:pot_fx_panel_small_knob_1, F.Cu at (133.9, 128.1)
- added REF**: sw_fx_panel_small, fx_synth_parts:sw_fx_panel_small, F.Cu at (138.8, 192.0)
- added REF**: pot_fx_panel_small_knob_2, fx_synth_parts:pot_fx_panel_small_knob_2, F.Cu at (103.4, 142.2)
- added REF**: pot_fx_panel_small_knob_2, fx_synth_parts:pot_fx_panel_small_knob_2, F.Cu at (103.4, 104.9)
- added REF**: MountingHole_3.2mm_M3_ISO14580_Pad, MountingHole:MountingHole_3.2mm_M3_ISO14580_Pad, F.Cu at (214.5, 43.5)
- added REF**: LED_D3.0mm, LED_THT:LED_D3.0mm, F.Cu at (125.2, 182.2)
- added REF**: pot_fx_panel_small_knob_2, fx_synth_parts:pot_fx_panel_small_knob_2, F.Cu at (103.4, 67.6)
- added REF**: sw_fx_panel_small, fx_synth_parts:sw_fx_panel_small, F.Cu at (130.0, 61.8)
- added REF**: pot_fx_panel_small_knob_1, fx_synth_parts:pot_fx_panel_small_knob_1, F.Cu at (165.3, 128.1)
- added REF**: jack_panel_small, fx_synth_parts:jack_panel_small, F.Cu at (150.3, 192.0)
- added REF**: pot_fx_panel_small_knob_2, fx_synth_parts:pot_fx_panel_small_knob_2, F.Cu at (103.4, 179.5)
- added REF**: pot_fx_panel_small_knob_2, fx_synth_parts:pot_fx_panel_small_knob_2, F.Cu at (195.4, 104.9)
- added REF**: pot_fx_panel_small_knob_2, fx_synth_parts:pot_fx_panel_small_knob_2, F.Cu at (195.3, 179.5)
- added REF**: sw_fx_panel_small, fx_synth_parts:sw_fx_panel_small, F.Cu at (130.0, 80.1)
- added REF**: pot_fx_panel_small_knob_2, fx_synth_parts:pot_fx_panel_small_knob_2, F.Cu at (195.4, 142.2)
- added REF**: MountingHole_3.2mm_M3_ISO14580_Pad, MountingHole:MountingHole_3.2mm_M3_ISO14580_Pad, F.Cu at (83.5, 206.0)
- added REF**: pot_fx_panel_small_knob_1, fx_synth_parts:pot_fx_panel_small_knob_1, F.Cu at (166.6, 190.2)
- added REF**: sw_fx_panel_small, fx_synth_parts:sw_fx_panel_small, F.Cu at (168.8, 61.8)
- added REF**: pot_fx_panel_small_knob_2, fx_synth_parts:pot_fx_panel_small_knob_2, F.Cu at (195.4, 67.6)
- added REF**: MountingHole_3.2mm_M3_ISO14580_Pad, MountingHole:MountingHole_3.2mm_M3_ISO14580_Pad, F.Cu at (83.5, 43.5)
- added REF**: sw_fx_panel_small, fx_synth_parts:sw_fx_panel_small, F.Cu at (130.0, 98.4)
- added REF**: sw_fx_panel_small, fx_synth_parts:sw_fx_panel_small, F.Cu at (168.8, 80.1)
- added locked: locked, , F.Cu at (119.8, 202.4)
- added locked: locked, , F.Cu at (179.3, 113.0)
- added locked: locked, , F.Cu at (179.3, 203.0)
- added locked: locked, , F.Cu at (179.4, 48.7)
- added locked: locked, , F.Cu at (119.8, 112.4)
- added locked: locked, , F.Cu at (119.9, 48.1)
Other:
- board size 100 x 205 mm -> 138 x 169.5 mm
- board text added: "LOW PASS FILTER"
- board text added: "MAIN"
- board text added: "OUT"
- board text added: "PWR"
- board text added: "SLICK"
- board text added: "SPK"
- board text added: "VOICE A"
- board text added: "VOICE B"
- board text added: "VOLTS"
- board text added: "VOLUME"
- board text added: "WACKY MOD"
- board text added: "ZANINESS"
- board text added: "off"
- board text added: "on"
- board text removed: "FREQ. MOD."
- board text removed: "WACKY TO WEIRD"
